File: Starbie_PCB/Starbie_PCB.kicad_pcb (KiCad board)
At the start: 2 copper layers, 64 x 80.5 mm, 7 parts, among them J1 Conn_01x04_Pin, J2 Conn_01x08_Pin, SW1 SW_Push, SW2 SW_Push, U1 DHT11, U2 XIAO-ESP32-C3-SMD

Commit message: Added day 3
Routing:
- net /GPI03: track 0.00 -> 111.2 mm
- net /GPI02: track 0.00 -> 88.2 mm
- net +3.3V: track 4.50 -> 90.8 mm, vias 0 -> 1
- net /SDA: track 0.00 -> 70.0 mm, vias 0 -> 2
- net /SCL: track 0.00 -> 63.0 mm
- net /DHT11 DATA: track 6.94 -> 26.2 mm
- added copper zone on B.Cu, net GND
- added copper zone on F.Cu, net GND
